Commit message: Complete simulation and wrote article.

File: urdf/common_macro.xacro (robot description, xacro)
@@ -1,4 +1,6 @@
 <?xml version="1.0"?>
-<robot name="mobile_robot_base" xmlns:xacro="http://www.ros.org/wiki/xacro">
+<robot name="common_macro" xmlns:xacro="http://www.ros.org/wiki/xacro">
+<!-- *********************************************************************** -->
+<!-- Константы -->
 <xacro:property name="PI" value="3.14"/>
 <!-- *********************************************************************** -->

File: urdf/corpus.xacro (robot description, xacro)
@@ -1,4 +1,4 @@
 <?xml version="1.0"?>
-<robot name="mobile_robot_base" xmlns:xacro="http://www.ros.org/wiki/xacro">
+<robot name="corpus" xmlns:xacro="http://www.ros.org/wiki/xacro">
 <!-- *********************************************************************** -->
 <xacro:include filename="$(find custom_ackermann_steering_controller_ros)/urdf/common_macro.xacro" />

File: urdf/main.xacro (robot description, xacro)
@@ -52,5 +52,5 @@
     <origin xyz="0.25 0.3 0" rpy="0 0 0"/>
     <axis xyz="0 0 1"/>
-    <limit lower="${-angle_wheel_limit}" upper="${angle_wheel_limit}" effort="1000" velocity="5"/>
+    <limit lower="${-angle_wheel_limit}" upper="${angle_wheel_limit}" effort="1000" velocity="1"/>
   </joint>
   <joint name="front_right_wheel_joint" type="revolute">
@@ -59,5 +59,5 @@
     <origin xyz="0.25 -0.3 0" rpy="0 0 0"/>
     <axis xyz="0 0 1"/>
-    <limit lower="${-angle_wheel_limit}" upper="${angle_wheel_limit}" effort="1000" velocity="5"/>
+    <limit lower="${-angle_wheel_limit}" upper="${angle_wheel_limit}" effort="1000" velocity="1"/>
   </joint>
   <!-- Суставы для соединения задних колес с корпусом (без поворота) -->

File: urdf/wheel.xacro (robot description, xacro)
@@ -1,4 +1,4 @@
 <?xml version="1.0"?>
-<robot name="mobile_robot_base" xmlns:xacro="http://www.ros.org/wiki/xacro">
+<robot name="wheel" xmlns:xacro="http://www.ros.org/wiki/xacro">
 <xacro:include filename="$(find custom_ackermann_steering_controller_ros)/urdf/common_macro.xacro" />
 <!-- *********************************************************************** -->
@@ -32,23 +32,3 @@
     </gazebo>
 </xacro:macro>
-<!-- *********************************************************************** -->
-<xacro:macro
-    name="wheel_hinge"
-    params="link_name">
-    <link name="${link_name}">
-        <visual>
-            <origin rpy="0 0 0" xyz="0 0 0"/>
-            <geometry>
-                <cylinder length="0.01" radius="0.025"/>
-            </geometry>
-            <material name="Green">
-                <color rgba="0.0 1.0 0.0 1.0"/>
-            </material>
-        </visual>
-        <xacro:cylinder_inertia m="1" r="0.1" h="0.1"/>
-    </link>
-    <gazebo reference ="${link_name}">
-        <material>Gazebo/Green</material>
-    </gazebo>
-</xacro:macro>
 </robot>
